Commit message: add lidar

File: railload_robot_description/urdf/railload_robot.urdf.xacro (robot description, xacro)
@@ -8,6 +8,6 @@
     <xacro:include filename="$(find railload_robot_description)/urdf/robot/base.urdf.xacro" />
     <xacro:include filename="$(find railload_robot_description)/urdf/robot/wheel.urdf.xacro" />
+    <xacro:include filename="$(find railload_robot_description)/urdf/sensors/VLP-16.urdf.xacro"/>
     <!-- <xacro:include filename="$(find railload_robot_description)/urdf/robot/differential_drive.gazebo.xacro" />
-    <xacro:include filename="$(find railload_robot_description)/urdf/sensors/lidar.urdf.xacro" />
     <xacro:include filename="$(find railload_robot_description)/urdf/sensors/d435.urdf.xacro" /> -->
     <!-- Robot Base -->
@@ -18,7 +18,8 @@
     <!-- <xacro:differential_drive_controller/> -->
     <!-- Lidars (Plugin) -->
-    <!-- <xacro:lidar>
-        <xacro:insert_block name="lidar_pose" />
-    </xacro:lidar> -->
+    <xacro:VLP-16 parent="base_link" name="velodyne" topic="/velodyne_points" hz="10" samples="440" gpu="false">
+        <!-- <xacro:insert_block name="lidar_pose" /> -->
+        <origin xyz="0 0 0.2" rpy="0 0 0" />
+    </xacro:VLP-16>
     <!-- IntelRealsense D435 (Plugin) -->
     <!-- <xacro:sensor_d435 parent="base_link" name="camera" use_nominal_extrinsics="$(arg use_nominal_extrinsics)">

File: railload_robot_description/urdf/railload_robot_properties.urdf.xacro (robot description, xacro)
@@ -10,5 +10,5 @@
     <!-- lidar property -->
     <xacro:property name="lidar_pose">
-        <origin xyz="0.679499999999998 0 0.236499999999997" rpy="1.5707963267949 0 0" />
+        <origin xyz="0 0 0.2" rpy="0 0 0" />
     </xacro:property>
     <!-- camera property -->

File: railload_robot_description/urdf/test.urdf (robot description, URDF)
Before this commit: robot railload_robot, 8 links, 7 joints
Links:
- added link velodyne, mass 0.01; collision sphere radius=0; visual mesh filename=package://velodyne_description/meshes/VLP16_scan.dae
- added link velodyne_base_link, mass 0.83; collision cylinder length=0.0717 radius=0.0516; visual mesh filename=package://velodyne_description/meshes/VLP16_base_1.dae
Joints:
- added joint velodyne_base_mount_joint: type fixed, parent base_link, child velodyne_base_link, origin xyz=0 0 0.2 rpy=0 0 0
- added joint velodyne_base_scan_joint: type fixed, parent velodyne_base_link, child velodyne, origin xyz=0 0 0.0377 rpy=0 0 0

Commit message: vlp16_gazebo

File: railload_robot_description/urdf/railload_robot.urdf.xacro (robot description, xacro)
@@ -8,7 +8,7 @@
     <xacro:include filename="$(find railload_robot_description)/urdf/robot/base.urdf.xacro" />
     <xacro:include filename="$(find railload_robot_description)/urdf/robot/wheel.urdf.xacro" />
-    <xacro:include filename="$(find railload_robot_description)/urdf/sensors/VLP-16.urdf.xacro"/>
-    <!-- <xacro:include filename="$(find railload_robot_description)/urdf/robot/differential_drive.gazebo.xacro" />
-    <xacro:include filename="$(find railload_robot_description)/urdf/sensors/d435.urdf.xacro" /> -->
+    <xacro:include filename="$(find railload_robot_description)/urdf/robot/differential_drive.gazebo.xacro" />
+    <xacro:include filename="$(find velodyne_description)/urdf/VLP-16.urdf.xacro"/>
+    <!-- <xacro:include filename="$(find railload_robot_description)/urdf/sensors/d435.urdf.xacro" /> -->
     <!-- Robot Base -->
     <xacro:base mass="${base_mass}"/>
@@ -16,9 +16,8 @@
     <xacro:wheel mass="${wheel_mass}"/>
     <!-- Differential Drive Controller (Plugin) -->
-    <!-- <xacro:differential_drive_controller/> -->
+    <xacro:differential_drive_controller/>
     <!-- Lidars (Plugin) -->
-    <xacro:VLP-16 parent="base_link" name="velodyne" topic="/velodyne_points" hz="10" samples="440" gpu="false">
-        <!-- <xacro:insert_block name="lidar_pose" /> -->
-        <origin xyz="0 0 0.2" rpy="0 0 0" />
+    <xacro:VLP-16 parent="base_link" name="velodyne" topic="/velodyne_points" hz="10" samples="440" gpu="true">
+        <xacro:insert_block name="lidar_pose" />
     </xacro:VLP-16>
     <!-- IntelRealsense D435 (Plugin) -->

Commit message: add railrobot_color

File: railload_robot_description/urdf/railload_robot.urdf.xacro (robot description, xacro)
@@ -9,4 +9,5 @@
     <xacro:include filename="$(find railload_robot_description)/urdf/robot/wheel.urdf.xacro" />
     <xacro:include filename="$(find railload_robot_description)/urdf/robot/differential_drive.gazebo.xacro" />
+    <xacro:include filename="$(find railload_robot_description)/urdf/robot/color.gazebo.xacro"/>
     <xacro:include filename="$(find velodyne_description)/urdf/VLP-16.urdf.xacro"/>
     <!-- <xacro:include filename="$(find railload_robot_description)/urdf/sensors/d435.urdf.xacro" /> -->
@@ -17,4 +18,6 @@
     <!-- Differential Drive Controller (Plugin) -->
     <xacro:differential_drive_controller/>
+    <!-- Gazebo Color -->
+    <xacro:gazebo_color/>
     <!-- Lidars (Plugin) -->
     <xacro:VLP-16 parent="base_link" name="velodyne" topic="/velodyne_points" hz="10" samples="440" gpu="true">

File: railload_robot_description/urdf/railload_robot_properties.urdf.xacro (robot description, xacro)
@@ -10,5 +10,5 @@
     <!-- lidar property -->
     <xacro:property name="lidar_pose">
-        <origin xyz="0 0 0.2" rpy="0 0 0" />
+        <origin xyz="0 0 0.5" rpy="0 0 0" />
     </xacro:property>
     <!-- camera property -->

File: railload_robot_description/urdf/robot/base.urdf.xacro (robot description, xacro)
@@ -18,4 +18,19 @@
             </collision>
             <xacro:box_inertial x="0.5" y="2.0" z="0.5" mass="5.0" />
+        </link>
+        <link name="lidar_pole">
+            <visual>
+                <origin xyz="0 0 0" rpy="0 0 0" />
+                <geometry>
+                    <cylinder radius="0.03" length="0.5"/>
+                </geometry>
+            </visual>
+            <collision>
+                <origin xyz="0 0 0" rpy="0 0 0" />
+                <geometry>
+                    <cylinder radius="0.03" length="0.5"/>
+                </geometry>
+            </collision>
+            <xacro:cylinder_inertial radius="0.03" length="0.5" mass="1.0" />
         </link>
         <!-- Front Body -->
@@ -69,4 +84,10 @@
             <origin xyz="0 0 0.3285" rpy="0 0 0"/>
         </joint>
+        <!-- Joint - base_link ~ lidar_pole -->
+        <joint name="base_link_to_lidar_pole" type="fixed">
+            <parent link="base_link"/>
+            <child link="lidar_pole"/>
+            <origin xyz="0 0 0.3" rpy="0 0 0"/>
+        </joint>
     </xacro:macro>
 </robot>
